File: builds/ergogen_xyz/pcbs/keyboard_v7.kicad_pcb (KiCad board)
At the start: 2 copper layers, 248 x 123.7 mm, 72 parts

Commit message: Phase 2: assembly hardware, wood cutting files, combined 3D render
- Add M2 mounting holes to PCB and outlines (4 corners per half)
- Add frame_with_holes outline for wood CNC/laser cutting
- Generate assembly.scad stacking all layers (frame, plates, PCB)
- Render assembly.png via OpenSCAD
- Update BOM with Phase 1 tenting mount and Phase 2 screws/standoffs
- Update render.md with assembly and wood cutting viewing instructions
- Update generate.sh with assembly generation and OpenSCAD render step

Co-Authored-By: Claude Opus 4.6 <noreply@anthropic.com>
Parts:
- added MH1: , MountingHole_M2, F.Cu at (0.28, -43.3)
- added MH2: , MountingHole_M2, F.Cu at (-5.57, 4.35)
- added MH3: , MountingHole_M2, F.Cu at (90.5, -33.5)
- added MH4: , MountingHole_M2, F.Cu at (80.6, 13.4)
