File: builds/ergogen_xyz/pcbs/keyboard_v7.kicad_pcb (KiCad board)
At the start: 2 copper layers, 258 x 131.8 mm, 76 parts

Commit message: Apply apple design fixes: bamboo frame, cork gaskets, ball joint, clevis pins
- Fix 1: Board fillet 2→8mm, frame fillet 3→10mm for smoother outline
- Fix 2: Bamboo plywood frame with 4mm wall (was 1mm walnut)
- Fix 3: Cork gasket layers (0.5mm each), total stack 3.8→4.8mm
- Fix 4: 7 mounting holes per half (was 4), heat-set brass inserts
- Fix 5: Turnbuckle cables with quick-release clevis pins (was carabiners)
- Fix 6: Ball joint hinge with thumb nut lock (was friction hinge)
- Fix 7: 301230 LiPo battery placement along board edge
- Updated BOM, render docs, and assembly 3D model

Co-Authored-By: Claude Opus 4.6 <noreply@anthropic.com>
Parts:
- added MH5: , MountingHole_M2, F.Cu at (50.3, -51.3)
- added MH6: , MountingHole_M2, F.Cu at (64.9, 29.5)
- added MH7: , MountingHole_M2, F.Cu at (57.5, 6.46)
Other:
- board size 258 x 131.8 mm -> 256.6 x 128.9 mm
